File: PCB/InstVirt.kicad_sch (KiCad schematic)
At the start: 58 parts, among them J1 Conn_01x20_Pin, J2 Conn_01x20_Pin, J3 Conn_01x08_Socket, J4 Conn_01x08_Socket, J5 Conn_01x08_Socket, J6 Conn_01x04, Q4 BC548, U1 4051, U10 PC817, U2 ULN2003, U3 PC817, U4 PC817, U5 PC817, U6 PC817, U7 PC817, U8 PC817, U9 PC817

Commit message: actualizacion pcb4
Parts:
- added C1, C2: 10uF, Capacitor_THT:CP_Radial_D5.0mm_P2.50mm, symbol Device:C_Polarized_US
- added D1: D_Zener, Diode_THT:D_DO-34_SOD68_P10.16mm_Horizontal, symbol Device:D_Zener
- added R42: 1K, Resistor_SMD:R_1206_3216Metric, symbol Device:R
- added R43: 1K, Resistor_THT:R_Axial_DIN0207_L6.3mm_D2.5mm_P10.16mm_Horizontal, symbol Device:R
- added R44, R45, R46, R47: 10K, Resistor_SMD:R_1206_3216Metric, symbol Device:R
- added R48: 180, Resistor_SMD:R_1206_3216Metric, symbol Device:R
- added R49: R, Resistor_SMD:R_1206_3216Metric, symbol Device:R
- added R50, R51: 1.8K, Resistor_THT:R_Axial_DIN0207_L6.3mm_D2.5mm_P10.16mm_Horizontal, symbol Device:R
- added RV1, RV2: 5k, Potentiometer_THT:Potentiometer_Bourns_3296W_Vertical, symbol Device:R_Potentiometer_Trim
- added RV3, RV4: 5K, Potentiometer_THT:Potentiometer_Bourns_3296W_Vertical, symbol Device:R_Potentiometer_Trim
- added U11, U12, U13: MCP6002-xMC, Package_DIP:DIP-8_W7.62mm_LongPads, symbol Amplifier_Operational:MCP6002-xMC
- J3, J5: footprint (none) -> Connector_PinHeader_2.54mm:PinHeader_1x08_P2.54mm_Vertical
- J4: footprint (none) -> Connector_PinSocket_2.54mm:PinSocket_1x08_P2.54mm_Vertical
- R1, R11, R13, R24, R27, R3, R31, R33, R35, R37, R39, R41, R5, R7, R9: footprint (none) -> Resistor_SMD:R_1206_3216Metric
- R10, R12, R14, R2, R25, R26, R28, R29, R32, R34, R36, R38, R4, R40, R6, R8: footprint (none) -> Resistor_THT:R_Axial_DIN0207_L6.3mm_D2.5mm_P10.16mm_Horizontal
- R15, R16: value R -> 1K; footprint (none) -> Resistor_SMD:R_1206_3216Metric
- R17, R18, R19, R20, R22, R30: value R10KΩ -> R1KΩ; footprint (none) -> Resistor_SMD:R_1206_3216Metric
- R21: value R10KΩ -> R1kΩ; footprint (none) -> Resistor_SMD:R_1206_3216Metric
- R23: value R10KΩ -> R1kKΩ; footprint (none) -> Resistor_SMD:R_1206_3216Metric
- U1: footprint (none) -> Package_DIP:DIP-16_W7.62mm_LongPads
- U2: footprint (none) -> Package_SO:SOP-16_4.4x10.4mm_P1.27mm
Connections:
- net B9ID2 is gone; now on net ID2: R26.2
- net A0O3: now also U2.6 (I6); no longer U2.5 (I5)
- net A15ID8: now also R41.1, U10.3; no longer R40.2
- net A1O4: now also U2.5 (I5); no longer U2.4 (I4)
- net A2O5: now also U2.4 (I4); no longer U2.3 (I3)
- net A3O6: now also U2.3 (I3); no longer U2.2 (I2)
- net A4O7: now also U2.2 (I2); no longer U2.1 (I1)
- net A5O8: now also U2.1 (I1); no longer R29.1
- net A6ADC1_IN6: now also U11.1, U11.2 (-); no longer U1.3 (X)
- net A7OPWM1: now also R49.2
- net B0OPWM2: now also R48.2
- net B3ID7: now also R39.1, U9.3
- net B4ID6: now also R37.1, U8.3; no longer R36.2
- net B5ID5: now also R35.1, U7.3; no longer R34.2
- net B6ID4: now also R33.1, U6.3; no longer R32.2
- net B7ID3: now also R31.1, U5.3; no longer R28.2
- net B8ID2: now also R27.1, U4.3
- net B9ID1: now also R24.1, U3.3; no longer R25.2
- net C14O1: now also R29.1; no longer U2.7 (I7)
- net C15O2: now also U2.7 (I7); no longer U2.6 (I6)
- net GND: now also C1.2, C2.2, D1.2 (A), R43.1, R46.2, R50.2, R51.2, RV1.2, RV1.3, RV2.3, U11.4 (V-), U11.9 (V-), U12.4 (V-), U12.9 (V-), U13.4 (V-), U13.9 (V-); no longer R16.1
- net ID1: now also R25.2; no longer R24.1, U3.3
- net ID2: no longer R27.1, U4.3
- net ID3: now also R28.2; no longer R31.1, U5.3
- net ID4: now also R32.2; no longer R33.1, U6.3
- net ID5: now also R34.2; no longer R35.1, U7.3
- net ID6: now also R36.2; no longer R37.1, U8.3
- net ID7: now also R38.2; no longer R39.1, U9.3
- net ID8: now also R40.2; no longer R41.1, U10.3
- net SD7: now also R22.1, U2.10 (O7)
- net VCC: now also R15.1, U11.8 (V+), U12.8 (V+), U13.8 (V+)
- net at R3.2, R4.2: now also U1.2 (X6); no longer U1.14 (X1)
- net at R10.2, R9.2: now also U1.15 (X2); no longer U1.1 (X4)
- net at R7.2, R8.2: now also U1.5 (X5); no longer U1.12 (X3)
- net at R5.2, R6.2: now also U1.4 (X7); no longer U1.15 (X2)
- net at J3.8 (Pin_8): now also R16.1
- net at R11.2, R12.2: now also U1.14 (X1); no longer U1.5 (X5)
- net at R13.2, R14.2: now also U1.13 (X0); no longer U1.2 (X6)
- net ADAPT: now reaches R1.2, R2.2
- net ADAPT: now also R44.1; no longer U1.13 (X0)
- net B1 renamed B1MUXA
- net B1MUXA: now also U1.11 (A)
- net B10 renamed B10MUXB
- net B10MUXB: now also U1.10 (B)
- net B11 renamed B11MUXC
- net B11MUXC: now also U1.9 (C)
- net B13MUXC renamed B13 
- net B13 : no longer U1.9 (C)
- net B14MUXB renamed B14 
- net B14 : no longer U1.10 (B)
- net B15MUXA renamed B15 
- net B15 : no longer U1.11 (A)
- new net: R44.2, R45.1, U12.3 (+)
- new net: R45.2, U12.6 (-), U12.7
- new net: R15.2, RV2.1, RV2.2, U12.5 (+)
- new net: RV3.1, RV3.2, U13.1
- new net: R50.1, RV3.3, U13.2 (-)
- new net: C1.1, R48.1, U13.3 (+)
- new net: R46.1, R47.2, U12.2 (-)
- new net: RV4.1, RV4.2, U13.7
- new net: R51.1, RV4.3, U13.6 (-)
- new net: R16.2, R43.2, U1.12 (X3)
- new net: C2.1, R49.1, U13.5 (+)
- new net: D1.1 (K), R42.2, RV1.1, U11.3 (+)
- new net: R42.1, U1.3 (X)
- new net SALID: R47.1, U1.1 (X4), U12.1
