File: PCB/InstVirt.kicad_sch (KiCad schematic)
At the start: 78 parts, among them J1 Conn_01x20_Pin, J2 Conn_01x20_Pin, J3 Conn_01x08_Socket, J4 Conn_01x08_Socket, J5 Conn_01x08_Socket, J6 Conn_01x04, Q4 BC548, U1 4051, U10 PC817, U11 MCP6002-xMC, U12 MCP6002-xMC, U13 MCP6002-xMC, U2 ULN2003, U3 PC817, U4 PC817, U5 PC817, U6 PC817, U7 PC817, U8 PC817, U9 PC817

Commit message: actualizacion pcb5
Parts:
- added BZ1: Buzzer, Buzzer_Beeper:MagneticBuzzer_ProSignal_ABI-010-RC, symbol Device:Buzzer
- added C10, C5, C6, C7: 10uF, Capacitor_THT:CP_Radial_D5.0mm_P2.50mm, symbol Device:C_Polarized_US
- added C3, C4, C8, C9: C, Capacitor_THT:C_Disc_D5.0mm_W2.5mm_P5.00mm, symbol Device:C
- added D2: LED, LED_THT:LED_D5.0mm, symbol Device:LED
- added J10, J11, J7, J8: Conn_01x01, Connector_PinSocket_2.54mm:PinSocket_1x01_P2.54mm_Vertical, symbol Connector_Generic:Conn_01x01
- added J12, J13: Conn_01x02, TerminalBlock_Phoenix:TerminalBlock_Phoenix_MKDS-1,5-2_1x02_P5.00mm_Horizontal, symbol Connector_Generic:Conn_01x02
- added J9: Conn_01x02, Connector_PinSocket_2.54mm:PinSocket_1x02_P2.54mm_Vertical, symbol Connector_Generic:Conn_01x02
- added JP1: Jumper_2_Bridged, Connector_PinSocket_2.54mm:PinSocket_1x02_P2.54mm_Vertical, symbol Jumper:Jumper_2_Bridged
- added R52: R, Resistor_THT:R_Axial_DIN0207_L6.3mm_D2.5mm_P10.16mm_Horizontal, symbol Device:R
- added U14, U15: L7805, Package_TO_SOT_THT:TO-220-3_Vertical, symbol Regulator_Linear:L7805
Connections:
- net ID1 is gone; now on net E1: R25.2
- net ID2 is gone; now on net E2: R26.2
- net ID3 is gone; now on net E3: R28.2
- net ID4 is gone; now on net E4: R32.2
- net ID5 is gone; now on net E5: R34.2
- net ID6 is gone; now on net E6: R36.2
- net ID7 is gone; now on net E8: R38.2
- net ID8 is gone; now on net E7: R40.2
- net +3.3V: now also C10.1, C9.1, J11.1 (Pin_1), JP1.1 (A), U15.3 (OUT)
- net B15 : now also BZ1.1 (-)
- net GND: now also J6.1 (Pin_1), BZ1.2 (+), C10.2, C3.2, C4.2, C5.2, C6.2, C7.2, C8.2, C9.2, J12.1 (Pin_1), J13.1 (Pin_1), J13.2 (Pin_2), R52.2, U14.2 (GND), U15.2 (GND)
- net GND2: now also J9.1 (Pin_1), J9.2 (Pin_2)
- net VCC: now also C4.1, C5.1, C7.1, C8.1, D2.2 (A), J10.1 (Pin_1), U14.3 (OUT), U15.1 (IN)
- net at RV3.1, RV3.2, U13.1: now also J7.1 (Pin_1)
- net at RV4.1, RV4.2, U13.7: now also J8.1 (Pin_1)
- net at J2.20 (Pin_20): now also JP1.2 (B)
- new net: D2.1 (K), R52.1
- new net +12V: C3.1, C6.1, J12.2 (Pin_2), U14.1 (IN)
Other:
- note added: "ALIMENTACION"
- note added: "COMUNICACION"
- note added: "SALIDA ANALOGA/ADAPTACION"
- moved on the sheet: C1, C2, D1, J1, J2, J4, J6, Q4, R15, R17, R18, R19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
