File: PCB/InstVirt.kicad_pcb (KiCad board)
At the start: 2 copper layers, 78 parts, among them J1 Conn_01x20_Pin, J2 Conn_01x20_Pin, J3 Conn_01x08_Socket, J4 Conn_01x08_Socket, J5 Conn_01x08_Socket, J6 Conn_01x04, Q4 BC548, U1 4051, U10 PC817, U11 MCP6002-xMC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

Commit message: actualizacion pcb5
Parts:
- added BZ1: Buzzer, Buzzer_Beeper:MagneticBuzzer_ProSignal_ABI-010-RC, F.Cu at (44.5, 156.1)
- added C10: 10uF, Capacitor_THT:CP_Radial_D5.0mm_P2.50mm, F.Cu at (107.8, 116.4)
- added C3: C, Capacitor_THT:C_Disc_D5.0mm_W2.5mm_P5.00mm, F.Cu at (94.8, 96.7)
- added C4: C, Capacitor_THT:C_Disc_D5.0mm_W2.5mm_P5.00mm, F.Cu at (94.8, 108.8)
- added C5: 10uF, Capacitor_THT:CP_Radial_D5.0mm_P2.50mm, F.Cu at (93.6, 103.0)
- added C6: 10uF, Capacitor_THT:CP_Radial_D5.0mm_P2.50mm, F.Cu at (93.5, 91.6)
- added C7: 10uF, Capacitor_THT:CP_Radial_D5.0mm_P2.50mm, F.Cu at (106.6, 107.5)
- added C8: C, Capacitor_THT:C_Disc_D5.0mm_W2.5mm_P5.00mm, F.Cu at (106.0, 101.1)
- added C9: C, Capacitor_THT:C_Disc_D5.0mm_W2.5mm_P5.00mm, F.Cu at (107.8, 122.1)
- added D2: LED, LED_THT:LED_D5.0mm, F.Cu at (83.8, 94.0)
- added J10: Conn_01x01, Connector_PinSocket_2.54mm:PinSocket_1x01_P2.54mm_Vertical, F.Cu at (92.4, 114.3)
- added J11: Conn_01x01, Connector_PinSocket_2.54mm:PinSocket_1x01_P2.54mm_Vertical, F.Cu at (105.3, 118.9)
- added J12: Conn_01x02, TerminalBlock_Phoenix:TerminalBlock_Phoenix_MKDS-1,5-2_1x02_P5.00mm_Horizontal, F.Cu at (109.3, 95.2)
- added J13: Conn_01x02, Connector_PinSocket_2.54mm:PinSocket_1x02_P2.54mm_Vertical, F.Cu at (97.8, 89.8)
- added J7: Conn_01x01, Connector_PinSocket_2.54mm:PinSocket_1x01_P2.54mm_Vertical, F.Cu at (35.3, 178.4)
- added J8: Conn_01x01, Connector_PinSocket_2.54mm:PinSocket_1x01_P2.54mm_Vertical, F.Cu at (61.9, 178.8)
- added J9: Conn_01x02, Connector_PinSocket_2.54mm:PinSocket_1x02_P2.54mm_Vertical, F.Cu at (106.5, 187.7)
- added JP1: Jumper_2_Bridged, Connector_PinSocket_2.54mm:PinSocket_1x02_P2.54mm_Vertical, F.Cu at (97.6, 146.9)
- added R52: R, Resistor_THT:R_Axial_DIN0207_L6.3mm_D2.5mm_P10.16mm_Horizontal, F.Cu at (79.3, 92.8)
- added U14: L7805, Package_TO_SOT_THT:TO-220-3_Vertical, F.Cu at (98.3, 97.3)
- added U15: L7805, Package_TO_SOT_THT:TO-220-3_Vertical, F.Cu at (100.5, 108.8)
- moved RV3 166.3 mm to (35.3, 172.1), turned to -90 degrees
- moved C1 164.7 mm to (41.1, 181.8), turned to -90 degrees
- moved U13 157.8 mm to (40.8, 169.7), turned to 0 degrees
- moved R50 157.5 mm to (39.5, 165.8), turned to 0 degrees
- moved C2 155.7 mm to (48.1, 181.2), turned to -90 degrees
- moved R49 155.6 mm to (45.4, 176.0), turned to 90 degrees
- moved R48 153.0 mm to (43.5, 167.2), turned to 90 degrees
- moved R43 151.8 mm to (35.6, 109.5), turned to 0 degrees
- moved R14 150.7 mm to (36.9, 106.4), turned to 0 degrees
- moved R12 149.7 mm to (38.2, 103.3), turned to 0 degrees
- moved R10 148.6 mm to (39.8, 99.9), turned to 0 degrees
- moved R16 147.0 mm to (42.1, 96.0), turned to -90 degrees
- moved R13 143.5 mm to (44.7, 96.0), turned to -90 degrees
- moved R51 143.3 mm to (58.2, 177.9), turned to 90 degrees
- moved RV4 143.1 mm to (53.3, 172.0), turned to 90 degrees
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Connections:
- J2 pad 20: unconnected-(J2-Pin_20-Pad20) -> Net-(J2-Pin_20)
- J6 pad 1: unconnected-(J6-Pin_1-Pad1) -> GND
- R25 pad 2: ID1 -> E1
- R26 pad 2: ID2 -> E2
- R28 pad 2: ID3 -> E3
- R32 pad 2: ID4 -> E4
- R34 pad 2: ID5 -> E5
- R36 pad 2: ID6 -> E6
- R38 pad 2: ID7 -> E8
- R40 pad 2: ID8 -> E7
Routing:
- net VCC: track 52.2 -> 238.5 mm, vias 0 -> 6
- net +3.3V: track 42.3 -> 173.3 mm
- net GND2: track 0.00 -> 41.4 mm
- net +12V: track 0.00 -> 23.4 mm
- net GND: track 0.00 -> 22.8 mm, vias 0 -> 8
- net Net-(R26-Pad1): track 0.00 -> 19.6 mm
- net Net-(R32-Pad1): track 0.00 -> 18.6 mm
- net Net-(R36-Pad1): track 0.00 -> 17.1 mm
- net Net-(R38-Pad1): track 0.00 -> 16.5 mm
- net E1: track 0.00 -> 15.4 mm
- net E2: track 0.00 -> 14.1 mm
- net B15 : track 0.00 -> 13.5 mm
- net E3: track 0.00 -> 11.5 mm
- net Net-(J8-Pin_1): track 7.44 -> 18.9 mm
- net E4: track 0.00 -> 10.3 mm
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- added copper zone on B.Cu, net +3.3V
- added copper zone on B.Cu, net GND
- added copper zone on B.Cu, net GND2
- added copper zone on B.Cu, net VCC
